File: 3.3V_DC_DC.kicad_sch (KiCad schematic)
At the start: 9 parts

Commit message: finish shcematic
Parts:
- added D7: 3.3, symbol Device:D_TVS
- L6: renamed from L?; LCSC (none) -> C57254
- gave numbers to parts that had none: 8
Connections:
- net +3.3V: now also D7.2 (A2)
- net GND: now also D7.1 (A1)
Changed lines of the file:
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@@
   (junction (at 59.055 50.165) (diameter 0) (color 0 0 0 0)
   )
+  (junction (at 191.135 53.975) (diameter 0) (color 0 0 0 0)
+  )
   (junction (at 76.835 50.165) (diameter 0) (color 0 0 0 0)
   )
@@
   (junction (at 172.085 78.105) (diameter 0) (color 0 0 0 0)
   )
+  (junction (at 191.135 78.105) (diameter 0) (color 0 0 0 0)
+  )
   (junction (at 91.44 50.165) (diameter 0) (color 0 0 0 0)
   )
@@
     (stroke (width 0) (type default) (color 0 0 0 0))
   )
+  (wire (pts (xy 191.135 70.485) (xy 191.135 78.105))
+    (stroke (width 0) (type default) (color 0 0 0 0))
+  )
   (wire (pts (xy 92.71 57.785) (xy 92.71 85.725))
     (stroke (width 0) (type default) (color 0 0 0 0))
@@
     (stroke (width 0) (type default) (color 0 0 0 0))
   )
-  (wire (pts (xy 179.705 78.105) (xy 172.085 78.105))
+  (wire (pts (xy 223.52 78.105) (xy 191.135 78.105))
     (stroke (width 0) (type default) (color 0 0 0 0))
   )
@@
     (stroke (width 0) (type default) (color 0 0 0 0))
   )
+  (wire (pts (xy 191.135 53.975) (xy 223.52 53.975))
+    (stroke (width 0) (type default) (color 0 0 0 0))
+  )
   (wire (pts (xy 143.51 53.975) (xy 143.51 56.515))
     (stroke (width 0) (type default) (color 0 0 0 0))
@@
     (stroke (width 0) (type default) (color 0 0 0 0))
   )
+  (wire (pts (xy 191.135 78.105) (xy 172.085 78.105))
+    (stroke (width 0) (type default) (color 0 0 0 0))
+  )
   (wire (pts (xy 121.285 57.785) (xy 121.285 68.58))
     (stroke (width 0) (type default) (color 0 0 0 0))
@@
     (stroke (width 0) (type default) (color 0 0 0 0))
   )
-  (wire (pts (xy 172.085 53.975) (xy 179.705 53.975))
+  (wire (pts (xy 191.135 53.975) (xy 191.135 62.865))
+    (stroke (width 0) (type default) (color 0 0 0 0))
+  )
+  (wire (pts (xy 172.085 53.975) (xy 191.135 53.975))
     (stroke (width 0) (type default) (color 0 0 0 0))
   )
@@
     (stroke (width 0) (type default) (color 0 0 0 0))
   )
-  (hierarchical_label "GND" (shape input) (at 179.705 78.105 0)
+  (hierarchical_label "GND" (shape input) (at 223.52 78.105 0)
     (effects (font (size 1.27 1.27)) (justify left))
   )
-  (hierarchical_label "+3.3V" (shape input) (at 179.705 53.975 0)
+  (hierarchical_label "+3.3V" (shape input) (at 223.52 53.975 0)
     (effects (font (size 1.27 1.27)) (justify left))
   )
@@
   (symbol (lib_id "power:GND") (at 172.085 85.725 0) (unit 1)
     (in_bom yes) (on_board yes) (fields_autoplaced)
-    (property "Reference" "#PWR?" (id 0) (at 172.085 92.075 0)
+    (property "Reference" "#PWR042" (id 0) (at 172.085 92.075 0)
       (effects (font (size 1.27 1.27)) hide)
     )
@@
   (symbol (lib_id "power:+3.3V") (at 172.085 47.625 0) (unit 1)
     (in_bom yes) (on_board yes) (fields_autoplaced)
-    (property "Reference" "#PWR?" (id 0) (at 172.085 51.435 0)
+    (property "Reference" "#PWR041" (id 0) (at 172.085 51.435 0)
       (effects (font (size 1.27 1.27)) hide)
     )
@@
   (symbol (lib_id "power:GND") (at 59.055 85.725 0) (unit 1)
     (in_bom yes) (on_board yes) (fields_autoplaced)
-    (property "Reference" "#PWR?" (id 0) (at 59.055 92.075 0)
+    (property "Reference" "#PWR037" (id 0) (at 59.055 92.075 0)
       (effects (font (size 1.27 1.27)) hide)
     )
@@
     (pin "1")
   )
+  (symbol (lib_id "Device:D_TVS") (at 191.135 66.675 90) (unit 1)
+    (in_bom yes) (on_board yes) (fields_autoplaced)
+    (property "Reference" "D7" (id 0) (at 193.675 65.4049 90)
+      (effects (font (size 1.27 1.27)) (justify right))
+    )
+    (property "Value" "3.3" (id 1) (at 193.675 67.9449 90)
+      (effects (font (size 1.27 1.27)) (justify right))
+    )
+    (property "Footprint" "" (id 2) (at 191.135 66.675 0)
+      (effects (font (size 1.27 1.27)) hide)
+    )
+    (property "Datasheet" "~" (id 3) (at 191.135 66.675 0)
+      (effects (font (size 1.27 1.27)) hide)
+    )
+    (pin "1")
+    (pin "2")
+  )
   (symbol (lib_id "Device:C") (at 172.085 68.58 0) (unit 1)
     (in_bom yes) (on_board yes) (fields_autoplaced)
-    (property "Reference" "C?" (id 0) (at 175.895 67.3099 0)
+    (property "Reference" "C31" (id 0) (at 175.895 67.3099 0)
       (effects (font (size 1.27 1.27)) (justify left))
     )
@@
   (symbol (lib_id "MT2492:MT2492") (at 106.045 51.435 0) (unit 1)
     (in_bom yes) (on_board yes) (fields_autoplaced)
-    (property "Reference" "U?" (id 0) (at 106.045 40.64 0))
+    (property "Reference" "U5" (id 0) (at 106.045 40.64 0))
     (property "Value" "MT2492" (id 1) (at 106.045 43.18 0))
     (property "Footprint" "Package_TO_SOT_SMD:SOT-23-6" (id 2) (at 106.045 62.865 0)
@@
   (symbol (lib_id "Device:C") (at 121.92 48.26 0) (unit 1)
     (in_bom yes) (on_board yes) (fields_autoplaced)
-    (property "Reference" "C?" (id 0) (at 125.73 46.9899 0)
+    (property "Reference" "C29" (id 0) (at 125.73 46.9899 0)
       (effects (font (size 1.27 1.27)) (justify left))
     )
@@
   (symbol (lib_id "Device:R") (at 157.48 60.325 0) (unit 1)
     (in_bom yes) (on_board yes) (fields_autoplaced)
-    (property "Reference" "R?" (id 0) (at 159.385 59.0549 0)
+    (property "Reference" "R22" (id 0) (at 159.385 59.0549 0)
       (effects (font (size 1.27 1.27)) (justify left))
     )
@@
   (symbol (lib_id "power:GND") (at 92.71 85.725 0) (unit 1)
     (in_bom yes) (on_board yes) (fields_autoplaced)
-    (property "Reference" "#PWR?" (id 0) (at 92.71 92.075 0)
+    (property "Reference" "#PWR039" (id 0) (at 92.71 92.075 0)
       (effects (font (size 1.27 1.27)) hide)
     )
@@
   (symbol (lib_id "power:GND") (at 76.835 85.725 0) (unit 1)
     (in_bom yes) (on_board yes) (fields_autoplaced)
-    (property "Reference" "#PWR?" (id 0) (at 76.835 92.075 0)
+    (property "Reference" "#PWR038" (id 0) (at 76.835 92.075 0)
       (effects (font (size 1.27 1.27)) hide)
     )
@@
   (symbol (lib_id "power:GND") (at 157.48 85.725 0) (unit 1)
     (in_bom yes) (on_board yes) (fields_autoplaced)
-    (property "Reference" "#PWR?" (id 0) (at 157.48 92.075 0)
+    (property "Reference" "#PWR040" (id 0) (at 157.48 92.075 0)
       (effects (font (size 1.27 1.27)) hide)
     )
@@
   (symbol (lib_id "Device:L") (at 136.525 53.975 90) (unit 1)
     (in_bom yes) (on_board yes)
-    (property "Reference" "L?" (id 0) (at 132.08 55.88 90))
+    (property "Reference" "L6" (id 0) (at 132.08 55.88 90))
     (property "Value" "SWPA6045S6R8MT" (id 1) (at 132.08 58.42 90))
     (property "Footprint" "" (id 2) (at 136.525 53.975 0)
       (effects (font (size 1.27 1.27)) hide)
     )
-    (property "Datasheet" "~" (id 3) (at 136.525 53.975 0)
+    (property "Datasheet" "https://datasheet.lcsc.com/lcsc/2110091630_Sunlord-SWPA6045S6R8MT_C57254.pdf" (id 3) (at 136.525 53.975 0)
+      (effects (font (size 1.27 1.27)) hide)
+    )
+    (property "LCSC" "C57254" (id 4) (at 136.525 53.975 90)
       (effects (font (size 1.27 1.27)) hide)
     )
@@
   (symbol (lib_id "Device:C_Polarized") (at 59.055 59.69 0) (unit 1)
     (in_bom yes) (on_board yes) (fields_autoplaced)
-    (property "Reference" "C?" (id 0) (at 62.865 57.5309 0)
+    (property "Reference" "C27" (id 0) (at 62.865 57.5309 0)
       (effects (font (size 1.27 1.27)) (justify left))
     )
@@
   (symbol (lib_id "Device:C") (at 76.835 59.055 0) (unit 1)
     (in_bom yes) (on_board yes) (fields_autoplaced)
-    (property "Reference" "C?" (id 0) (at 80.645 57.7849 0)
+    (property "Reference" "C28" (id 0) (at 80.645 57.7849 0)
       (effects (font (size 1.27 1.27)) (justify left))
     )
@@
   (symbol (lib_id "Device:R") (at 157.48 76.835 0) (unit 1)
     (in_bom yes) (on_board yes) (fields_autoplaced)
-    (property "Reference" "R?" (id 0) (at 159.385 75.5649 0)
+    (property "Reference" "R23" (id 0) (at 159.385 75.5649 0)
       (effects (font (size 1.27 1.27)) (justify left))
     )
@@
   (symbol (lib_id "Device:C") (at 143.51 60.325 0) (unit 1)
     (in_bom yes) (on_board yes) (fields_autoplaced)
-    (property "Reference" "C?" (id 0) (at 146.685 59.0549 0)
-      (effects (font (size 1.27 1.27)) (justify left))
-    )
+    (property "Reference" "C30" (id 0) (at 146.685 59.0549 0)
+      (effects (font (size 1.27 1.27)) (justify left))
+    )

Commit message: Add some more footprints
Parts:
- C27, C28, C30, C31: footprint (none) -> Capacitor_SMD:C_0603_1608Metric_Pad1.08x0.95mm_HandSolder
- C29: value 0.1u -> 100n; footprint (none) -> Capacitor_SMD:C_0603_1608Metric_Pad1.08x0.95mm_HandSolder
- R22, R23: footprint (none) -> Resistor_SMD:R_0603_1608Metric_Pad0.98x0.95mm_HandSolder
Changed lines of the file:
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@@
       (effects (font (size 1.27 1.27)) (justify left))
     )
-    (property "Footprint" "" (id 2) (at 173.0502 72.39 0)
+    (property "Footprint" "Capacitor_SMD:C_0603_1608Metric_Pad1.08x0.95mm_HandSolder" (id 2) (at 173.0502 72.39 0)
       (effects (font (size 1.27 1.27)) hide)
     )
@@
       (effects (font (size 1.27 1.27)) (justify left))
     )
-    (property "Value" "0.1u" (id 1) (at 125.73 49.5299 0)
+    (property "Value" "100n" (id 1) (at 125.73 49.5299 0)
       (effects (font (size 1.27 1.27)) (justify left))
     )
-    (property "Footprint" "" (id 2) (at 122.8852 52.07 0)
+    (property "Footprint" "Capacitor_SMD:C_0603_1608Metric_Pad1.08x0.95mm_HandSolder" (id 2) (at 122.8852 52.07 0)
       (effects (font (size 1.27 1.27)) hide)
     )
@@
       (effects (font (size 1.27 1.27)) (justify left))
     )
-    (property "Footprint" "" (id 2) (at 155.702 60.325 90)
+    (property "Footprint" "Resistor_SMD:R_0603_1608Metric_Pad0.98x0.95mm_HandSolder" (id 2) (at 155.702 60.325 90)
       (effects (font (size 1.27 1.27)) hide)
     )
@@
       (effects (font (size 1.27 1.27)) (justify left))
     )
-    (property "Footprint" "" (id 2) (at 60.0202 63.5 0)
+    (property "Footprint" "Capacitor_SMD:C_0603_1608Metric_Pad1.08x0.95mm_HandSolder" (id 2) (at 60.0202 63.5 0)
       (effects (font (size 1.27 1.27)) hide)
     )
@@
       (effects (font (size 1.27 1.27)) (justify left))
     )
-    (property "Footprint" "" (id 2) (at 77.8002 62.865 0)
+    (property "Footprint" "Capacitor_SMD:C_0603_1608Metric_Pad1.08x0.95mm_HandSolder" (id 2) (at 77.8002 62.865 0)
       (effects (font (size 1.27 1.27)) hide)
     )
@@
       (effects (font (size 1.27 1.27)) (justify left))
     )
-    (property "Footprint" "" (id 2) (at 155.702 76.835 90)
+    (property "Footprint" "Resistor_SMD:R_0603_1608Metric_Pad0.98x0.95mm_HandSolder" (id 2) (at 155.702 76.835 90)
       (effects (font (size 1.27 1.27)) hide)
     )
@@
       (effects (font (size 1.27 1.27)) (justify left))
     )
-    (property "Footprint" "" (id 2) (at 144.4752 64.135 0)
+    (property "Footprint" "Capacitor_SMD:C_0603_1608Metric_Pad1.08x0.95mm_HandSolder" (id 2) (at 144.4752 64.135 0)
       (effects (font (size 1.27 1.27)) hide)
     )

Commit message: Add even more footprints
Parts:
- D7: footprint (none) -> Diode_SMD:D_SMA-SMB_Universal_Handsoldering
Changed lines of the file:
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@@
       (effects (font (size 1.27 1.27)) (justify right))
     )
-    (property "Footprint" "" (id 2) (at 191.135 66.675 0)
+    (property "Footprint" "Diode_SMD:D_SMA-SMB_Universal_Handsoldering" (id 2) (at 191.135 66.675 0)
       (effects (font (size 1.27 1.27)) hide)
     )

Commit message: basic ETH layout
Parts:
- L6: footprint (none) -> SWPA6045S6R8MT:SWPA6045S6R8MT
Changed lines of the file:
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@@
     (property "Reference" "L6" (id 0) (at 132.08 55.88 90))
     (property "Value" "SWPA6045S6R8MT" (id 1) (at 132.08 58.42 90))
-    (property "Footprint" "" (id 2) (at 136.525 53.975 0)
+    (property "Footprint" "SWPA6045S6R8MT:SWPA6045S6R8MT" (id 2) (at 136.525 53.975 0)
       (effects (font (size 1.27 1.27)) hide)
     )

Commit message: layout fixes
Parts:
- C27: footprint Capacitor_SMD:C_0603_1608Metric_Pad1.08x0.95mm_HandSolder -> Capacitor_Tantalum_SMD:CP_EIA-7343-30_AVX-N_Pad2.25x2.55mm_HandSolder
Changed lines of the file:
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@@
       (effects (font (size 1.27 1.27)) (justify left))
     )
-    (property "Footprint" "Capacitor_SMD:C_0603_1608Metric_Pad1.08x0.95mm_HandSolder" (id 2) (at 60.0202 63.5 0)
+    (property "Footprint" "Capacitor_Tantalum_SMD:CP_EIA-7343-30_AVX-N_Pad2.25x2.55mm_HandSolder" (id 2) (at 60.0202 63.5 0)
       (effects (font (size 1.27 1.27)) hide)
     )

Commit message: Add more LCSC markings, change to electrolytic caps :
Parts:
- C27: footprint Capacitor_Tantalum_SMD:CP_EIA-7343-30_AVX-N_Pad2.25x2.55mm_HandSolder -> Capacitor_SMD:CP_Elec_6.3x7.7; LCSC (none) -> C4747974
- C28: LCSC (none) -> C92487
- C29: LCSC (none) -> C282519
- C30: LCSC (none) -> C376775
- C31: LCSC (none) -> C140782
- R22: LCSC (none) -> C5140983
- R23: LCSC (none) -> C2907001
- U5: LCSC (none) -> C89358
Changed lines of the file:
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@@
+      (effects (font (size 1.27 1.27)) hide)
+    )
+    (property "LCSC" "C140782" (id 4) (at 172.085 68.58 0)
       (effects (font (size 1.27 1.27)) hide)
     )
@@
     )
     (property "Datasheet" "https://datasheet.lcsc.com/lcsc/1810262207_XI-AN-Aerosemi-Tech-MT2492_C89358.pdf" (id 3) (at 106.045 62.865 0)
+      (effects (font (size 1.27 1.27)) hide)
+    )
+    (property "LCSC" "C89358" (id 4) (at 106.045 51.435 0)
       (effects (font (size 1.27 1.27)) hide)
     )
@@
       (effects (font (size 1.27 1.27)) hide)
     )
+    (property "LCSC" "C282519" (id 4) (at 121.92 48.26 0)
+      (effects (font (size 1.27 1.27)) hide)
+    )
     (pin "1")
     (pin "2")
@@
     )
     (property "Datasheet" "~" (id 3) (at 157.48 60.325 0)
+      (effects (font (size 1.27 1.27)) hide)
+    )
+    (property "LCSC" "C5140983" (id 4) (at 157.48 60.325 0)
       (effects (font (size 1.27 1.27)) hide)
     )
@@
       (effects (font (size 1.27 1.27)) (justify left))
     )
-    (property "Footprint" "Capacitor_Tantalum_SMD:CP_EIA-7343-30_AVX-N_Pad2.25x2.55mm_HandSolder" (id 2) (at 60.0202 63.5 0)
+    (property "Footprint" "Capacitor_SMD:CP_Elec_6.3x7.7" (id 2) (at 60.0202 63.5 0)
       (effects (font (size 1.27 1.27)) hide)
     )
@@
       (effects (font (size 1.27 1.27)) hide)
     )
+    (property "LCSC" "C4747974" (id 4) (at 59.055 59.69 0)
+      (effects (font (size 1.27 1.27)) hide)
+    )
     (pin "1")
     (pin "2")
@@
       (effects (font (size 1.27 1.27)) hide)
     )
+    (property "LCSC" "C92487" (id 4) (at 76.835 59.055 0)
+      (effects (font (size 1.27 1.27)) hide)
+    )
     (pin "1")
     (pin "2")
@@
       (effects (font (size 1.27 1.27)) hide)
     )
+    (property "LCSC" "C2907001" (id 4) (at 157.48 76.835 0)
+      (effects (font (size 1.27 1.27)) hide)
+    )
     (pin "1")
     (pin "2")
@@
       (effects (font (size 1.27 1.27)) hide)
     )
+    (property "LCSC" "C376775" (id 4) (at 143.51 60.325 0)
+      (effects (font (size 1.27 1.27)) hide)
+    )

Commit message: Update kicad files
Other:
- note added: "Przetwornica działa, trzeba uważać żeby nie zjarać scalaka"
