File: ESP32.kicad_sch (KiCad schematic)
At the start: 1 part

Commit message: finish shcematic
Parts:
- added C32: 47u, symbol Device:C
- added C33: 22u, symbol Device:C
- added C34: 100n, symbol Device:C
- gave numbers to parts that had none: 1
Connections:
- net GND: now reaches U6.1 (GND), U6.15 (GND), U6.38 (GND), U6.39 (GND)
- net GND: now also C32.2, C33.2, C34.2
- net EMAC_RXD0: now reaches U6.10 (IO25)
- net EMAC_RXD1: now reaches U6.11 (IO26)
- net EMAC_CRS_DV: now reaches U6.12 (IO27)
- net IO14: now reaches U6.13 (IO14)
- net IO12: now reaches U6.14 (IO12)
- net IO13: now reaches U6.16 (IO13)
- net +3V3: now reaches U6.2 (VDD)
- net +3V3: now also C32.1
- net IO15: now reaches U6.23 (IO15)
- net IO2: now reaches U6.24 (IO2)
- net IO0: now reaches U6.25 (IO0)
- net IO4: now reaches U6.26 (IO4)
- net EMAC_MDC: now reaches U6.27 (IO16)
- net EMAC_MDIO: now reaches U6.28 (IO17)
- net IO5: now reaches U6.29 (IO5)
- net ESP_EN: now reaches U6.3 (EN)
- net ESP_EN: now also C33.1, C34.1
- net IO18: now reaches U6.30 (IO18)
- net EMAC_TXD0: now reaches U6.31 (IO19)
- net EMAC_TX_EN: now reaches U6.33 (IO21)
- net RX: now reaches U6.34 (RXD0/IO3)
- net TX: now reaches U6.35 (TXD0/IO1)
- net EMAC_TXD1: now reaches U6.36 (IO22)
- net IO23: now reaches U6.37 (IO23)
- net IO34: now reaches U6.6 (IO34)
- net IO35: now reaches U6.7 (IO35)
- net IO32: now reaches U6.8 (IO32)
- net IO33: now reaches U6.9 (IO33)

Commit message: feat: add more LCSC symbols
Parts:
- U6: LCSC (none) -> C473012
Changed lines of the file:
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@@
+      (effects (font (size 1.27 1.27)) hide)
+    )
+    (property "LCSC" "C473012" (id 4) (at 144.78 93.98 0)
       (effects (font (size 1.27 1.27)) hide)
     )

Commit message: Add some more footprints
Parts:
- C32, C33, C34: footprint (none) -> Capacitor_SMD:C_0603_1608Metric_Pad1.08x0.95mm_HandSolder
Changed lines of the file:
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@@
       (effects (font (size 1.27 1.27)) (justify left))
     )
-    (property "Footprint" "" (id 2) (at 115.9002 73.025 0)
+    (property "Footprint" "Capacitor_SMD:C_0603_1608Metric_Pad1.08x0.95mm_HandSolder" (id 2) (at 115.9002 73.025 0)
       (effects (font (size 1.27 1.27)) hide)
     )
@@
       (effects (font (size 1.27 1.27)) (justify left))
     )
-    (property "Footprint" "" (id 2) (at 105.7402 73.025 0)
+    (property "Footprint" "Capacitor_SMD:C_0603_1608Metric_Pad1.08x0.95mm_HandSolder" (id 2) (at 105.7402 73.025 0)
       (effects (font (size 1.27 1.27)) hide)
     )
@@
       (effects (font (size 1.27 1.27)) (justify left))
     )
-    (property "Footprint" "" (id 2) (at 89.2302 106.68 0)
+    (property "Footprint" "Capacitor_SMD:C_0603_1608Metric_Pad1.08x0.95mm_HandSolder" (id 2) (at 89.2302 106.68 0)
       (effects (font (size 1.27 1.27)) hide)
     )

Commit message: Finish layout
Connections:
- net IO32: no longer names the net of U6.8 (IO32)
- net IO33: no longer names the net of U6.9 (IO33)
- net IO34: no longer names the net of U6.6 (IO34)
- net IO35: no longer names the net of U6.7 (IO35)
- no-connect marks 0 -> 4
Other:
- note added: "GPIO 0 (must be LOW to enter boot mode) GPIO 2 (must be floating or LOW during boot) GPIO 4. GPIO 5 (must be HIGH during boot) GPIO 12 (must be LOW during boot) GPIO 15 (must be HIGH during boot)"
- note added: "GPIOs 34 to 39 are GPIs - input only pins"
- note added: "IO32 IO33 are connected to the crystal. Docs say you can't use these 2x pins as GPIO unless you desolder some stuff on the module."
Changed lines of the file:
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@@
   (junction (at 104.775 63.5) (diameter 0) (color 0 0 0 0)
   )
+  (no_connect (at 160.02 119.38))
+  (no_connect (at 160.02 121.92))
+  (no_connect (at 160.02 116.84))
+  (no_connect (at 160.02 114.3))
   (wire (pts (xy 104.775 73.025) (xy 104.775 76.2))
     (stroke (width 0) (type default) (color 0 0 0 0))
@@
     (stroke (width 0) (type default) (color 0 0 0 0))
   )
-  (wire (pts (xy 160.02 119.38) (xy 163.195 119.38))
-    (stroke (width 0) (type default) (color 0 0 0 0))
-  )
   (wire (pts (xy 104.775 63.5) (xy 114.935 63.5))
     (stroke (width 0) (type default) (color 0 0 0 0))
@@
   )
   (wire (pts (xy 160.02 71.12) (xy 163.195 71.12))
-    (stroke (width 0) (type default) (color 0 0 0 0))
-  )
-  (wire (pts (xy 160.02 116.84) (xy 163.195 116.84))
     (stroke (width 0) (type default) (color 0 0 0 0))
   )
@@
     (stroke (width 0) (type default) (color 0 0 0 0))
   )
-  (wire (pts (xy 160.02 114.3) (xy 163.195 114.3))
-    (stroke (width 0) (type default) (color 0 0 0 0))
-  )
   (wire (pts (xy 160.02 83.82) (xy 163.195 83.82))
     (stroke (width 0) (type default) (color 0 0 0 0))
@@
     (stroke (width 0) (type default) (color 0 0 0 0))
   )
-  (wire (pts (xy 160.02 121.92) (xy 163.195 121.92))
-    (stroke (width 0) (type default) (color 0 0 0 0))
-  )
   (wire (pts (xy 88.265 94.615) (xy 88.265 99.06))
     (stroke (width 0) (type default) (color 0 0 0 0))
@@
     (stroke (width 0) (type default) (color 0 0 0 0))
   )
+  (text "IO32 IO33 are connected to the crystal. Docs say you can't use these 2x pins as GPIO unless you desolder some stuff on the module.\n"
+    (at 184.15 83.82 0)
+    (effects (font (size 1.27 1.27)) (justify left bottom))
+  )
+  (text "GPIOs 34 to 39 are GPIs - input only pins" (at 184.15 80.645 0)
+    (effects (font (size 1.27 1.27)) (justify left bottom))
+  )
+  (text "GPIO 0 (must be LOW to enter boot mode)\nGPIO 2 (must be floating or LOW during boot)\nGPIO 4.\nGPIO 5 (must be HIGH during boot)\nGPIO 12 (must be LOW during boot)\nGPIO 15 (must be HIGH during boot)"
+    (at 184.15 75.565 0)
+    (effects (font (size 1.27 1.27)) (justify left bottom))
+  )
   (hierarchical_label "IO13" (shape input) (at 163.195 81.28 0)
-    (effects (font (size 1.27 1.27)) (justify left))
-  )
-  (hierarchical_label "IO32" (shape input) (at 163.195 114.3 0)
-    (effects (font (size 1.27 1.27)) (justify left))
-  )
-  (hierarchical_label "IO34" (shape input) (at 163.195 119.38 0)
     (effects (font (size 1.27 1.27)) (justify left))
   )
@@
     (effects (font (size 1.27 1.27)) (justify left))
   )
-  (hierarchical_label "IO35" (shape input) (at 163.195 121.92 0)
-    (effects (font (size 1.27 1.27)) (justify left))
-  )
   (hierarchical_label "TX" (shape input) (at 163.195 66.04 0)
     (effects (font (size 1.27 1.27)) (justify left))
@@
     (effects (font (size 1.27 1.27)) (justify left))
   )
-  (hierarchical_label "IO33" (shape input) (at 163.195 116.84 0)
-    (effects (font (size 1.27 1.27)) (justify left))
-  )

Commit message: Add testpoints, jumpers
Parts:
- added R33: 10k, Resistor_SMD:R_0603_1608Metric_Pad0.98x0.95mm_HandSolder, symbol Device:R
Connections:
- net ESP_EN: now also R33.2
- new net +3.3V: R33.1
Changed lines of the file:
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@@
 (kicad_sch (version 20211123) (generator eeschema)
   (paper "A4")
+  (junction (at 120.015 63.5) (diameter 0) (color 0 0 0 0)
+  )
   (junction (at 114.935 63.5) (diameter 0) (color 0 0 0 0)
   )
@@
     (stroke (width 0) (type default) (color 0 0 0 0))
   )
-  (wire (pts (xy 114.935 63.5) (xy 129.54 63.5))
+  (wire (pts (xy 114.935 63.5) (xy 120.015 63.5))
     (stroke (width 0) (type default) (color 0 0 0 0))
   )
@@
     (stroke (width 0) (type default) (color 0 0 0 0))
   )
+  (wire (pts (xy 120.015 47.625) (xy 120.015 50.8))
+    (stroke (width 0) (type default) (color 0 0 0 0))
+  )
+  (wire (pts (xy 120.015 58.42) (xy 120.015 63.5))
+    (stroke (width 0) (type default) (color 0 0 0 0))
+  )
   (wire (pts (xy 160.02 66.04) (xy 163.195 66.04))
     (stroke (width 0) (type default) (color 0 0 0 0))
   )
   (wire (pts (xy 88.265 94.615) (xy 88.265 99.06))
+    (stroke (width 0) (type default) (color 0 0 0 0))
+  )
+  (wire (pts (xy 120.015 63.5) (xy 129.54 63.5))
     (stroke (width 0) (type default) (color 0 0 0 0))
   )
@@
       (effects (font (size 1.27 1.27)) hide)
     )
+    (pin "1")
+    (pin "2")
+  )
+  (symbol (lib_id "power:+3.3V") (at 120.015 47.625 0) (unit 1)
+    (in_bom yes) (on_board yes) (fields_autoplaced)
+    (property "Reference" "#PWR0109" (id 0) (at 120.015 51.435 0)
+      (effects (font (size 1.27 1.27)) hide)
+    )
+    (property "Value" "+3.3V" (id 1) (at 120.015 41.91 0))
+    (property "Footprint" "" (id 2) (at 120.015 47.625 0)
+      (effects (font (size 1.27 1.27)) hide)
+    )
+    (property "Datasheet" "" (id 3) (at 120.015 47.625 0)
+      (effects (font (size 1.27 1.27)) hide)
+    )
+    (pin "1")
+  )
+  (symbol (lib_id "Device:R") (at 120.015 54.61 0) (unit 1)
+    (in_bom yes) (on_board yes) (fields_autoplaced)
+    (property "Reference" "R33" (id 0) (at 121.92 53.3399 0)
+      (effects (font (size 1.27 1.27)) (justify left))
+    )
+    (property "Value" "10k" (id 1) (at 121.92 55.8799 0)
+      (effects (font (size 1.27 1.27)) (justify left))
+    )
+    (property "Footprint" "Resistor_SMD:R_0603_1608Metric_Pad0.98x0.95mm_HandSolder" (id 2) (at 118.237 54.61 90)
+      (effects (font (size 1.27 1.27)) hide)
+    )
+    (property "Datasheet" "~" (id 3) (at 120.015 54.61 0)
+      (effects (font (size 1.27 1.27)) hide)
+    )

Commit message: Add more LCSC markings, change to electrolytic caps :
Parts:
- C32: LCSC (none) -> C140782
- C33: LCSC (none) -> C59461
- C34: LCSC (none) -> C282519
- R33: LCSC (none) -> C2930027
Changed lines of the file:
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@@
+      (effects (font (size 1.27 1.27)) hide)
+    )
+    (property "LCSC" "C282519" (id 4) (at 114.935 69.215 0)
       (effects (font (size 1.27 1.27)) hide)
     )
@@
     )
     (property "Datasheet" "~" (id 3) (at 120.015 54.61 0)
+      (effects (font (size 1.27 1.27)) hide)
+    )
+    (property "LCSC" "C2930027" (id 4) (at 120.015 54.61 0)
       (effects (font (size 1.27 1.27)) hide)
     )
@@
     )
     (property "Datasheet" "~" (id 3) (at 104.775 69.215 0)
+      (effects (font (size 1.27 1.27)) hide)
+    )
+    (property "LCSC" "C59461" (id 4) (at 104.775 69.215 0)
       (effects (font (size 1.27 1.27)) hide)
     )
@@
       (effects (font (size 1.27 1.27)) hide)
     )
+    (property "LCSC" "C140782" (id 4) (at 88.265 102.87 0)
+      (effects (font (size 1.27 1.27)) hide)
+    )
