File: wiegand_interface.kicad_sch (KiCad schematic)
At the start: 10 parts, among them U7 LTV-827S, U8 LTV-827S

Commit message: Remove non-standard resistor
Parts:
- R29, R31: value 190 -> 186
Changed lines of the file:
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@@
       (effects (font (size 1.27 1.27)) (justify left))
     )
-    (property "Value" "190" (id 1) (at 175.895 123.1899 0)
+    (property "Value" "186" (id 1) (at 175.895 123.1899 0)
       (effects (font (size 1.27 1.27)) (justify left))
     )
@@
       (effects (font (size 1.27 1.27)) (justify left))
     )
-    (property "Value" "190" (id 1) (at 146.05 123.1899 0)
+    (property "Value" "186" (id 1) (at 146.05 123.1899 0)
       (effects (font (size 1.27 1.27)) (justify left))
     )

Commit message: fixup wrong resistor values
Parts:
- R29, R31: value 186 -> 180
Changed lines of the file:
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@@
       (effects (font (size 1.27 1.27)) (justify left))
     )
-    (property "Value" "186" (id 1) (at 175.895 123.1899 0)
+    (property "Value" "180" (id 1) (at 175.895 123.1899 0)
       (effects (font (size 1.27 1.27)) (justify left))
     )
@@
       (effects (font (size 1.27 1.27)) (justify left))
     )
-    (property "Value" "186" (id 1) (at 146.05 123.1899 0)
+    (property "Value" "180" (id 1) (at 146.05 123.1899 0)
       (effects (font (size 1.27 1.27)) (justify left))
     )

Commit message: Add some more footprints
Parts:
- R26, R27, R28, R29, R30, R31: footprint (none) -> Resistor_SMD:R_0603_1608Metric_Pad0.98x0.95mm_HandSolder
Changed lines of the file:
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@@
       (effects (font (size 1.27 1.27)) (justify left))
     )
-    (property "Footprint" "" (id 2) (at 91.567 83.82 90)
+    (property "Footprint" "Resistor_SMD:R_0603_1608Metric_Pad0.98x0.95mm_HandSolder" (id 2) (at 91.567 83.82 90)
       (effects (font (size 1.27 1.27)) hide)
     )
@@
       (effects (font (size 1.27 1.27)) (justify left))
     )
-    (property "Footprint" "" (id 2) (at 116.332 83.82 90)
+    (property "Footprint" "Resistor_SMD:R_0603_1608Metric_Pad0.98x0.95mm_HandSolder" (id 2) (at 116.332 83.82 90)
       (effects (font (size 1.27 1.27)) hide)
     )
@@
       (effects (font (size 1.27 1.27)) (justify left))
     )
-    (property "Footprint" "" (id 2) (at 142.367 79.375 90)
+    (property "Footprint" "Resistor_SMD:R_0603_1608Metric_Pad0.98x0.95mm_HandSolder" (id 2) (at 142.367 79.375 90)
       (effects (font (size 1.27 1.27)) hide)
     )
@@
       (effects (font (size 1.27 1.27)) (justify left))
     )
-    (property "Footprint" "" (id 2) (at 172.212 121.92 90)
+    (property "Footprint" "Resistor_SMD:R_0603_1608Metric_Pad0.98x0.95mm_HandSolder" (id 2) (at 172.212 121.92 90)
       (effects (font (size 1.27 1.27)) hide)
     )
@@
       (effects (font (size 1.27 1.27)) (justify left))
     )
-    (property "Footprint" "" (id 2) (at 172.212 79.375 90)
+    (property "Footprint" "Resistor_SMD:R_0603_1608Metric_Pad0.98x0.95mm_HandSolder" (id 2) (at 172.212 79.375 90)
       (effects (font (size 1.27 1.27)) hide)
     )
@@
       (effects (font (size 1.27 1.27)) (justify left))
     )
-    (property "Footprint" "" (id 2) (at 142.367 121.92 90)
-      (effects (font (size 1.27 1.27)) hide)
-    )
+    (property "Footprint" "Resistor_SMD:R_0603_1608Metric_Pad0.98x0.95mm_HandSolder" (id 2) (at 142.367 121.92 90)
+      (effects (font (size 1.27 1.27)) hide)
+    )

Commit message: Add even more footprints
Parts:
- D8, D9: footprint (none) -> Diode_SMD:D_SMA-SMB_Universal_Handsoldering
Changed lines of the file:
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@@
     (property "Reference" "D8" (id 0) (at 151.13 108.585 0))
     (property "Value" "5V5" (id 1) (at 151.13 111.125 0))
-    (property "Footprint" "" (id 2) (at 151.13 114.3 0)
+    (property "Footprint" "Diode_SMD:D_SMA-SMB_Universal_Handsoldering" (id 2) (at 151.13 114.3 0)
       (effects (font (size 1.27 1.27)) hide)
     )
@@
     (property "Reference" "D9" (id 0) (at 180.975 108.585 0))
     (property "Value" "5V5" (id 1) (at 180.975 111.125 0))
-    (property "Footprint" "" (id 2) (at 180.975 114.3 0)
+    (property "Footprint" "Diode_SMD:D_SMA-SMB_Universal_Handsoldering" (id 2) (at 180.975 114.3 0)
       (effects (font (size 1.27 1.27)) hide)
     )

Commit message: Add more LCSC markings, change to electrolytic caps :
Parts:
- R26, R27: LCSC (none) -> C2974027
- R28, R30: value 140 -> 10k; LCSC (none) -> C2930027
- R29, R31: LCSC (none) -> C5140972
- U7, U8: LCSC (none) -> C22112
Changed lines of the file:
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@@
+      (effects (font (size 1.27 1.27)) hide)
+    )
+    (property "LCSC" "C2974027" (id 4) (at 93.345 83.82 0)
       (effects (font (size 1.27 1.27)) hide)
     )
@@
     )
     (property "Datasheet" "http://www.us.liteon.com/downloads/LTV-817-827-847.PDF" (id 3) (at 129.54 78.105 0)
+      (effects (font (size 1.27 1.27)) hide)
+    )
+    (property "LCSC" "C22112" (id 4) (at 115.57 98.425 90)
       (effects (font (size 1.27 1.27)) hide)
     )
@@
       (effects (font (size 1.27 1.27)) hide)
     )
+    (property "LCSC" "C2974027" (id 4) (at 118.11 83.82 0)
+      (effects (font (size 1.27 1.27)) hide)
+    )
     (pin "1")
     (pin "2")
@@
       (effects (font (size 1.27 1.27)) (justify left))
     )
-    (property "Value" "140" (id 1) (at 146.05 80.6449 0)
+    (property "Value" "10k" (id 1) (at 146.05 80.6449 0)
       (effects (font (size 1.27 1.27)) (justify left))
     )
@@
     )
     (property "Datasheet" "~" (id 3) (at 144.145 79.375 0)
+      (effects (font (size 1.27 1.27)) hide)
+    )
+    (property "LCSC" "C2930027" (id 4) (at 144.145 79.375 0)
       (effects (font (size 1.27 1.27)) hide)
     )
@@
       (effects (font (size 1.27 1.27)) hide)
     )
+    (property "LCSC" "C5140972" (id 4) (at 173.99 121.92 0)
+      (effects (font (size 1.27 1.27)) hide)
+    )
     (pin "1")
     (pin "2")
@@
       (effects (font (size 1.27 1.27)) (justify left))
     )
-    (property "Value" "140" (id 1) (at 176.53 80.6449 0)
+    (property "Value" "10k" (id 1) (at 176.53 80.6449 0)
       (effects (font (size 1.27 1.27)) (justify left))
     )
@@
       (effects (font (size 1.27 1.27)) hide)
     )
+    (property "LCSC" "C2930027" (id 4) (at 173.99 79.375 0)
+      (effects (font (size 1.27 1.27)) hide)
+    )
     (pin "1")
     (pin "2")
@@
     )
     (property "Datasheet" "http://www.us.liteon.com/downloads/LTV-817-827-847.PDF" (id 3) (at 104.775 77.47 0)
+      (effects (font (size 1.27 1.27)) hide)
+    )
+    (property "LCSC" "C22112" (id 4) (at 90.805 97.79 90)
       (effects (font (size 1.27 1.27)) hide)
     )
@@
       (effects (font (size 1.27 1.27)) hide)
     )
+    (property "LCSC" "C22112" (id 4) (at 176.53 98.425 90)
+      (effects (font (size 1.27 1.27)) hide)
+    )
     (pin "1")
     (pin "2")
@@
       (effects (font (size 1.27 1.27)) hide)
     )
+    (property "LCSC" "C5140972" (id 4) (at 144.145 121.92 0)
+      (effects (font (size 1.27 1.27)) hide)
+    )
     (pin "1")
     (pin "2")
@@
   )
   (symbol (lib_id "power:GND") (at 154.305 93.98 0) (unit 1)
-    (in_bom yes) (on_board yes) (fields_autoplaced)
+    (in_bom yes) (on_board yes)
     (property "Reference" "#PWR060" (id 0) (at 154.305 100.33 0)
       (effects (font (size 1.27 1.27)) hide)
     )
-    (property "Value" "GND" (id 1) (at 154.305 99.06 0))
+    (property "Value" "GND" (id 1) (at 158.75 95.25 0))
     (property "Footprint" "" (id 2) (at 154.305 93.98 0)
       (effects (font (size 1.27 1.27)) hide)
