File: wiegand_interface.kicad_sch (KiCad schematic)
At the start: 15 parts, among them U10 EL3H7-G, U11 EL3H7-G, U7 EL3H7-G, U8 EL3H7-G, U9 EL3H7-G

Commit message: misc updates, extend board
Parts:
- added D18, D19: PESD5V0L1BA, Diode_SMD:D_SOD-323, symbol Device:D_TVS
- added R38, R42: 10k, Resistor_SMD:R_0603_1608Metric_Pad0.98x0.95mm_HandSolder, symbol Device:R
- added R43, R44: 470, Resistor_SMD:R_0603_1608Metric_Pad0.98x0.95mm_HandSolder, symbol Device:R
- added U13, U14: EL3H7-G, Package_SO:SSOP-4_4.4x2.6mm_P1.27mm, symbol Isolator:Optocoupler_DC_PhotoNPN_AKEC
Connections:
- net AUX_INP_12V: now also R43.2, R44.2
- net DAT0: now also R38.2
- net DAT1: now also R42.2
- net GND: now also U13.3, U14.3
- net GND2: now also D11.2 (A2), D12.2 (A2), U7.3, U9.3
- net READER_BUZZER: now also D11.1 (A1), U7.4; no longer D11.2 (A2), U7.3
- net READER_LED: now also D12.1 (A1), U9.4; no longer D12.2 (A2), U9.3
- net AUX_INP_GND renamed AUX_INP1_GND
- net AUX_INP_INV renamed AUX_INP1_INV
- removed net EXT_PWR: D11.1 (A1), D12.1 (A1), U7.4, U9.4
- new net: D18.2 (A2), R43.1, U13.1
- new net: D19.2 (A2), R44.1, U14.1
- new net +3.3V: R38.1, R42.1
- new net AUX_INP2_GND: D18.1 (A1), U13.2
- new net AUX_INP2_INV: U13.4
- new net AUX_INP3_GND: D19.1 (A1), U14.2
- new net AUX_INP3_INV: U14.4
Other:
- note added: "LED/Buzzer zwiera się do masy"
- note added: "Pull-ups needed, because ESP doesn't allow internal pullups on IO34 and IO35"
- moved on the sheet: D11, D12, D8, D9, R26, R27, R29, R31, U10, U7, U8, U9

Commit message: Zamkonator rev 1.3
Parts:
- renumbered D12 to D13, D11 to D14, D8 to D15, D9 to D16, D14 to D17, R26 to R34, R27 to R35, R42 to R36, R29 to R37, R31 to R39, R39 to R40, R43 to R41, R44 to R42, U8 to U11, U11 to U12, U9 to U8, U7 to U9
