File: USB_to_serial.kicad_sch (KiCad schematic)
At the start: 20 parts, among them Q2 SS8050G, Q3 SS8050G, U15 CH9102F

Commit message: Rev 1.3, BOM optimizations
Parts:
- C40, C41: value 100n -> 100n 100V
Changed lines of the file:
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@@
 			)
 		)
-		(property "Value" "100n"
+		(property "Value" "100n 100V"
 			(at 100.33 44.45 90)
 			(show_name no)
@@
 			)
 		)
-		(property "Value" "100n"
+		(property "Value" "100n 100V"
 			(at 100.33 55.88 90)
 			(show_name no)
